Commit message: add sylinder pointing at origin

File: rsc/husky/husky.urdf (robot description, URDF)
Before this commit: robot husky_robot, 11 links, 10 joints
Joints:
- joint imu_joint: origin xyz=0.25 0 0.509 rpy=0 0 3.14159 -> xyz=0.25 0 0.3 rpy=0 0 0

Commit message: first_success_with_6.5s

File: rsc/husky/husky.urdf (robot description, URDF)
Before this commit: robot husky_robot, 11 links, 10 joints
Joints:
- joint imu_joint: origin xyz=0.25 0 0.3 rpy=0 0 0 -> xyz=0.25 0 0.5 rpy=0 0 0
